File: Projeto1/Prototipage_aula2.kicad_sch (KiCad schematic)
At the start: 14 parts, among them J2 284697-E, J3 Conn_01x07_Pin, J4 Conn_01x06_Pin, U1 BMI088

Commit message: update
Parts:
- J3: footprint Connector_PinSocket_2.54mm:PinSocket_1x07_P2.54mm_Vertical -> Connector_PinHeader_2.54mm:PinHeader_1x07_P2.54mm_Vertical
- J4: footprint Connector_PinSocket_2.54mm:PinSocket_1x06_P2.54mm_Vertical -> Connector_PinHeader_2.54mm:PinHeader_1x06_P2.54mm_Vertical
Changed lines of the file:
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@@
 			)
 		)
-		(property "Footprint" "Connector_PinSocket_2.54mm:PinSocket_1x06_P2.54mm_Vertical"
+		(property "Footprint" "Connector_PinHeader_2.54mm:PinHeader_1x06_P2.54mm_Vertical"
 			(at 154.94 151.13 0)
 			(effects
@@
 	)
 	(symbol
+		(lib_id "Connector:Conn_01x07_Pin")
+		(at 104.14 151.13 90)
+		(unit 1)
+		(exclude_from_sim no)
+		(in_bom yes)
+		(on_board yes)
+		(dnp no)
+		(fields_autoplaced yes)
+		(property "Reference" "J3"
+			(at 104.14 153.67 90)
+			(effects
+				(font
+					(size 1.27 1.27)
+				)
+			)
+		)
+		(property "Value" "Conn_01x07_Pin"
+			(at 104.14 156.21 90)
+			(effects
+				(font
+					(size 1.27 1.27)
+				)
+				(hide yes)
+			)
+		)
+		(property "Footprint" "Connector_PinHeader_2.54mm:PinHeader_1x07_P2.54mm_Vertical"
+			(at 104.14 151.13 0)
+			(effects
+				(font
+					(size 1.27 1.27)
+				)
+				(hide yes)
+			)
+		)
+		(property "Datasheet" "~"
+			(at 104.14 151.13 0)
+			(effects
+				(font
+					(size 1.27 1.27)
+				)
+				(hide yes)
+			)
+		)
+		(property "Description" "Generic connector, single row, 01x07, script generated"
+			(at 104.14 151.13 0)
+			(effects
+				(font
+					(size 1.27 1.27)
+				)
+				(hide yes)
+			)
+		)
+		(pin "1"
+		)
+		(pin "2"
+		)
+		(pin "6"
+		)
+		(pin "7"
+		)
+		(pin "4"
+		)
+		(pin "3"
+		)
+		(pin "5"
+		)
+		(instances
+			(project ""
+				(path "/78a6c22b-848d-43da-b85b-7e3cc2070649"
+					(reference "J3")
+					(unit 1)
+				)
+			)
+		)
+	)
+	(symbol
 		(lib_id "Device:R")
 		(at 97.79 46.99 0)
@@
 					(unit 1)
 				)
-			)
-		)
-	)
-	(symbol
-		(lib_id "Connector:Conn_01x07_Pin")
-		(at 104.14 151.13 90)
-		(unit 1)
-		(exclude_from_sim no)
-		(in_bom yes)
-		(on_board yes)
-		(dnp no)
-		(fields_autoplaced yes)
-		(property "Reference" "J3"
-			(at 104.14 153.67 90)
-			(effects
-				(font
-					(size 1.27 1.27)
-				)
-			)
-		)
-		(property "Value" "Conn_01x07_Pin"
-			(at 104.14 156.21 90)
-			(effects
-				(font
-					(size 1.27 1.27)
-				)
-				(hide yes)
-			)
-		)
-		(property "Footprint" "Connector_PinSocket_2.54mm:PinSocket_1x07_P2.54mm_Vertical"
-			(at 104.14 151.13 0)
-			(effects
-				(font
-					(size 1.27 1.27)
-				)
-				(hide yes)
-			)
-		)
-		(property "Datasheet" "~"
-			(at 104.14 151.13 0)
-			(effects
-				(font
-					(size 1.27 1.27)
-				)
-				(hide yes)
-			)
-		)
-		(property "Description" "Generic connector, single row, 01x07, script generated"
-			(at 104.14 151.13 0)
-			(effects
-				(font
-					(size 1.27 1.27)
-				)
-				(hide yes)
-			)
-		)
-		(pin "1"
-		)
-		(pin "3"
-		)
-		(pin "5"
-		)
-		(pin "2"
-		)
-		(pin "6"
-		)
-		(pin "7"
-		)
-		(pin "4"
-		)
-		(instances
-			(project ""
-				(path "/78a6c22b-848d-43da-b85b-7e3cc2070649"
-					(reference "J3")
-					(unit 1)
-				)

Commit message: ahhhhhhhhhhhhhhh
Parts:
- removed D1: APT1608LZGCK, Prototipagem_Lib:LED_APT1608LZGCK, symbol Prototipagem_Lib:APT1608LZGCK
- removed J2: 284697-E, Prototipagem_Lib:284697E, symbol Prototipagem_Lib:284697-E
- removed U1: BMI088, Prototipagem_Lib:PQFN50P450X300X100-16N, symbol Prototipagem_Lib:BMI088
- added D1: APT1608LZGCK, APT1608LZGCK:LED_APT1608LZGCK, symbol Lib:APT1608LZGCK
- added J1: 284697-E, 284697E, symbol Lib:284697-E
- added U2: BMI088, BMI088:PQFN50P450X300X100-16N, symbol Lib:BMI088
Connections:
- net +3V3: now also J1.1, U2.11 (VDDIO), U2.3 (VDD)
- net CSB1: now also U2.14 (CSB1)
- net CSB2: now also U2.5 (CSB2)
- net GND: now also D1.1, J1.5 (S1), J1.7 (S3), U2.4 (GNDA), U2.6 (GNDIO)
- net INT1: now also U2.16 (INT1)
- net INT2: now also U2.1 (INT2)
- net INT3: now also U2.12 (INT3)
- net INT4: now also U2.13 (INT4)
- net PS: now also U2.7 (PS)
- net SCL: now also J1.3, U2.8 (SCL/SCK)
- net SDA: now also J1.2, U2.9 (SDA/SDI)
- net SDO1: now also U2.15 (SDO1)
- net SDO2: now also U2.10 (SDO2)
- net at R3.2: now also D1.2
- new net: J1.4, J1.6 (S2), J1.8 (S4)
