File: Projeto1/Prototipage_aula2.kicad_sch (KiCad schematic)
At the start: 14 parts, among them J1 284697-E, J3 Conn_01x07_Pin, J4 Conn_01x06_Pin, U1 BMI088

Commit message: lol
Parts:
- added H1, H2, H3: ~, symbol Lib:Screw
- added PH1, PH2, PH3: ~, symbol Lib:Via_Screw
- J3: footprint Connector_PinHeader_2.54mm:PinHeader_1x07_P2.54mm_Vertical -> Connector_PinHeader_2.00mm:PinHeader_1x07_P2.00mm_Vertical
- J4: footprint Connector_PinHeader_2.54mm:PinHeader_1x06_P2.54mm_Vertical -> Connector_PinHeader_2.00mm:PinHeader_1x06_P2.00mm_Vertical
Connections:
- net GND: now also J1.4, J1.6 (S2), J1.8 (S4)

Commit message: Projeto1 Acabado
Other:
- note added: "PCB holders"
Changed lines of the file:
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@@
 	(paper "A4")
 	(rectangle
-		(start 37.592 94.488)
-		(end 68.58 158.75)
+		(start 37.592 93.98)
+		(end 68.58 160.02)
 		(stroke
 			(width 0)
@@
 	)
 	(rectangle
-		(start 81.534 94.488)
-		(end 184.404 159.004)
+		(start 81.534 93.98)
+		(end 184.404 160.02)
 		(stroke
 			(width 0)
@@
 		)
 	)
+	(rectangle
+		(start 208.28 93.98)
+		(end 261.62 160.02)
+		(stroke
+			(width 0)
+			(type dash)
+		)
+		(fill
+			(type none)
+		)
+	)
+	(text "PCB holders"
+		(exclude_from_sim no)
+		(at 216.662 98.044 0)
+		(effects
+			(font
+				(size 1.27 1.27)
+			)
+		)
+	)
