File: Projeto1/_autosave-Prototipage_aula2.kicad_sch (KiCad schematic)
At the start: 14 parts, among them J1 284697-E, J3 Conn_01x07_Pin, J4 Conn_01x06_Pin, U1 BMI088

Commit message: update
Connections:
- net GND: now also J1.4, J1.6 (S2), J1.8 (S4)
Changed lines of the file:
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@@
+	)
+	(junction
+		(at 64.77 60.96)
+		(diameter 0)
+		(color 0 0 0 0)
 	)
 	(junction
@@
 	(wire
 		(pts
+			(xy 64.77 60.96) (xy 68.58 60.96)
+		)
+		(stroke
+			(width 0)
+			(type default)
+		)
+	)
+	(wire
+		(pts
 			(xy 97.79 50.8) (xy 97.79 53.34)
 		)
@@
 		)
 		(stroke
+			(width 0)
+			(type default)
+		)
+	)
+	(wire
+		(pts
+			(xy 68.58 60.96) (xy 68.58 69.85)
+		)
+		(stroke
