File: Projeto1/Prototipage_aula2.kicad_pcb (KiCad board)
At the start: 2 copper layers, 25 x 30 mm, 14 parts, among them J2 284697-E, J3 Conn_01x07_Pin, J4 Conn_01x06_Pin, U1 BMI088

Commit message: update
Parts:
- J3: footprint Connector_PinSocket_2.54mm:PinSocket_1x07_P2.54mm_Vertical -> Connector_PinHeader_2.54mm:PinHeader_1x07_P2.54mm_Vertical
- J4: footprint Connector_PinSocket_2.54mm:PinSocket_1x06_P2.54mm_Vertical -> Connector_PinHeader_2.54mm:PinHeader_1x06_P2.54mm_Vertical
- moved J4 1.96 mm to (150.0, 72.5)
- moved J3 1.16 mm to (130.5, 70.5)
- moved C2 1.12 mm to (139.9, 91.5), turned to 180 degrees
- moved R5 0.69 mm to (134.0, 84.0), turned to 180 degrees
- moved D1 0.18 mm to (139.7, 74.0), turned to 180 degrees
Routing:
- net +3V3: track 0.00 -> 43.2 mm
- net SDA: track 0.00 -> 23.7 mm
- net Net-(D1-Pad1): track 0.00 -> 2.73 mm
- added copper zone on B.Cu, net GND
- added copper zone on F.Cu, net GND

Commit message: update
Routing:
- net SDO2: track 0.00 -> 31.8 mm
- net (no net): track 0.00 -> 30.3 mm
- net SCL: track 0.00 -> 24.6 mm, vias 0 -> 3
- net INT3: track 0.00 -> 23.1 mm, vias 0 -> 1
- net SDO1: track 0.00 -> 17.3 mm
- net INT2: track 0.00 -> 14.1 mm, vias 0 -> 1
- net INT1: track 0.00 -> 13.2 mm, vias 0 -> 1
- net CSB2: track 0.00 -> 13.2 mm, vias 0 -> 1
- net SDA: track 23.7 -> 35.7 mm, vias 0 -> 2
- net PS: track 0.00 -> 11.9 mm, vias 0 -> 1
- net CSB1: track 0.00 -> 11.6 mm
- net INT4: track 0.00 -> 11.1 mm

Commit message: ahhhhhhhhhhhhhhh
Parts:
- removed D1: APT1608LZGCK, Prototipagem_Lib:LED_APT1608LZGCK
- removed J2: 284697-E, Prototipagem_Lib:284697E
- removed U1: BMI088, Prototipagem_Lib:PQFN50P450X300X100-16N

Commit message: update
Parts:
- added D2: APT1608LZGCK, Lib_footprint:LED_APT1608LZGCK, F.Cu at (139.5, 74.0)
- added J1: 284697-E, Lib_footprint:284697E, F.Cu at (140.1, 68.0)
- added U1: BMI088, Lib_footprint:PQFN50P450X300X100-16N, F.Cu at (139.9, 87.5)
- moved C2 3.60 mm to (143.5, 91.0), turned to 0 degrees
- moved R3 1.00 mm to (139.4, 75.5)
- moved R6 0.99 mm to (146.0, 82.0)
- moved J4 0.50 mm to (149.5, 72.5)
- moved R1 0.50 mm to (139.4, 77.5)
- moved R7 0.50 mm to (139.4, 81.5)
Routing:
- net (no net): track 30.3 -> 0.00 mm
- net SCL: track 24.6 -> 49.6 mm
- net SDA: track 35.7 -> 41.2 mm
- net PS: track 11.9 -> 16.7 mm
- net GND: track 0.00 -> 3.00 mm, vias 0 -> 15
- net SDO2: track 31.8 -> 33.5 mm
- net INT4: track 11.1 -> 12.6 mm
- net Net-(D2-Pad2): track 2.73 -> 2.03 mm
- net CSB2: track 13.2 -> 12.7 mm

Commit message: lol
Parts:
- added REF**: MountingHole_3.2mm_M3_ISO14580_Pad, MountingHole:MountingHole_3.2mm_M3_ISO14580_Pad, F.Cu at (149.0, 66.0)
- added REF**: MountingHole_3.2mm_M3_ISO14580_Pad, MountingHole:MountingHole_3.2mm_M3_ISO14580_Pad, F.Cu at (149.0, 89.0)
- added REF**: MountingHole_3.2mm_M3_ISO14580_Pad, MountingHole:MountingHole_3.2mm_M3_ISO14580_Pad, F.Cu at (131.0, 66.0)
- J3: footprint Connector_PinHeader_2.54mm:PinHeader_1x07_P2.54mm_Vertical -> Connector_PinHeader_2.00mm:PinHeader_1x07_P2.00mm_Vertical
- J4: footprint Connector_PinHeader_2.54mm:PinHeader_1x06_P2.54mm_Vertical -> Connector_PinHeader_2.00mm:PinHeader_1x06_P2.00mm_Vertical
- moved C2 2.50 mm to (141.0, 91.0)
Routing:
- net SDO2: track 33.5 -> 18.6 mm, vias 0 -> 2
- net SCL: track 49.6 -> 44.2 mm
- net CSB1: track 11.5 -> 15.2 mm, vias 0 -> 1
- net INT4: track 12.6 -> 16.1 mm
- net GND: track 3.00 -> 6.21 mm, vias 15 -> 13
- net +3V3: track 43.0 -> 41.2 mm
- net INT1: track 13.2 -> 14.8 mm
- net CSB2: track 12.7 -> 14.2 mm
- net SDO1: track 17.3 -> 15.8 mm
- net SDA: track 41.2 -> 39.9 mm
- net INT2: track 14.1 -> 15.1 mm
- net PS: track 16.7 -> 17.7 mm
Other:
- outline, holes or cut-outs redrawn

Commit message: Projeto1 Acabado
Parts:
- moved R4 1.03 mm to (133.7, 79.5)
- moved R6 0.50 mm to (146.0, 81.5)
Routing:
- net GND: track 6.21 -> 13.3 mm
- net SDA: track 39.9 -> 41.3 mm
- net CSB1: track 15.2 -> 16.1 mm
- net SDO1: track 15.8 -> 16.7 mm
- net CSB2: track 14.2 -> 13.3 mm
Other:
- board text added: "3V3"
- board text added: "CSB1"
- board text added: "CSB2"
- board text added: "GND"
- board text added: "I2C"
- board text added: "INT1"
- board text added: "INT2"
- board text added: "INT3"
- board text added: "INT4"
- board text added: "PS"
- board text added: "R5"
- board text added: "SCL"
- board text added: "SDA"
- board text added: "SDO1"
- board text added: "SDO2"
