File: Projeto2/Projeto2.kicad_sch (KiCad schematic)
At the start: 0 parts

Commit message: step by step
Parts:
- added C02, C04: 10n, Capacitor_SMD:C_0805_2012Metric_Pad1.18x1.45mm_HandSolder, symbol Device:C_Small
- added C03: 1u, Capacitor_SMD:C_0805_2012Metric_Pad1.18x1.45mm_HandSolder, symbol Device:C_Small
- added C05, C06: 47p, Capacitor_SMD:C_0805_2012Metric_Pad1.18x1.45mm_HandSolder, symbol Device:C_Small
- added C07: 4u7, Capacitor_SMD:C_0603_1608Metric_Pad1.08x0.95mm_HandSolder, symbol Device:C_Small
- added C08, C09, C11, C13, C16, C19, C22, C25, C28: 100n, Capacitor_SMD:C_0603_1608Metric_Pad1.08x0.95mm_HandSolder, symbol Device:C_Small
- added C1: 2u2, Capacitor_SMD:C_0805_2012Metric_Pad1.18x1.45mm_HandSolder, symbol Device:C_Small
- added C10, C15, C20, C23, C26, C29: 10u, Capacitor_SMD:C_0805_2012Metric_Pad1.18x1.45mm_HandSolder, symbol Device:C_Small
- added C12, C14, C17, C18, C21, C24, C27: 10n, Capacitor_SMD:C_0603_1608Metric_Pad1.08x0.95mm_HandSolder, symbol Device:C_Small
- added D1: LED_BLUE, symbol Lib:LED_BLUE
- added J1, J2: Conn_02x03_Odd_Even, symbol Lib:Conn_02x03_Odd_Even
- added L1: FerriteBead_Small, Inductor_SMD:L_0603_1608Metric_Pad1.05x0.95mm_HandSolder, symbol Device:FerriteBead_Small
- added L2: 0.2n, Inductor_SMD:L_0402_1005Metric_Pad0.77x0.64mm_HandSolder, symbol Device:L
- added P1: 10118194-0001LF, Lib_fp:AMPHENOL_10118194-0001LF, symbol Lib:10118194-0001LF
- added R01, R2: 1k, Resistor_SMD:R_0603_1608Metric_Pad0.98x0.95mm_HandSolder, symbol Device:R_US
- added R03, R04: 27, Resistor_SMD:R_0603_1608Metric_Pad0.98x0.95mm_HandSolder, symbol Device:R_US
- added U1: TPS79633DCQR, Lib_fp:VREG_TPS79633DCQR, symbol Lib:TPS79633DCQR
- added U2: FT231XS-R, Package_SO:SSOP-20_3.9x8.7mm_P0.635mm, symbol Lib:FT231XS-R
- added U3: PIC32MZ1024EFE064-E/PT, TQFP64_PT_MCH, symbol Lib:PIC32MZ1024EFE064-E_PT
Connections:
- new net: C04.1, L1.1, P1.1 (VCC)
- new net: C05.1, P1.2 (D-), R03.1
- new net: C06.1, P1.3 (D+), R04.1
- new net: J1.1 (Pin_1), R01.1
- new net: C03.1, J2.1 (Pin_1), U1.4 (OUT)
- new net: C09.1, J2.3 (Pin_3), R2.2, U2.13 (3V3OUT), U2.14 (~{RESET}), U2.3 (VCCIO)
- new net: C02.1, U1.5 (NR/FB)
- new net: D1.2 (A), R2.1
- new net: R04.2, U2.11 (USBDP)
- new net: R03.2, U2.12 (USBDM)
- new net +3V3: C10.2, C11.2, C12.2, C13.1, C14.1, C15.2, C16.2, C17.2, C18.1, C19.1, C20.1, C21.2, C22.2, C23.2, C24.2, C25.2, C26.2, C27.2, C28.2, C29.2, J2.2 (Pin_2), J2.4 (Pin_4), J2.6 (Pin_6), L2.1, L2.2, U3.19 (AVDD), U3.26 (VDD), U3.34 (VUSB3V3), U3.39 (VDD), U3.54 (VDD), U3.60 (VDD), U3.8 (VDD)
- new net +3V3AUX: J2.5 (Pin_5)
- new net +5V: C1.1, J1.2 (Pin_2), J1.4 (Pin_4), J1.6 (Pin_6), U1.1 (EN), U1.2 (IN)
- new net +5V0USB: C07.1, C08.1, J1.5 (Pin_5), L1.2, U2.15 (VCC)
- new net +5VAUX: J1.3 (Pin_3)
- new net D+: U3.37 (D+)
- new net D-: U3.36 (D-)
- new net GND: C02.2, C03.2, C04.2, C05.2, C06.2, C07.2, C08.2, C09.2, C1.2, C10.1, C11.1, C12.1, C13.2, C14.2, C15.1, C16.1, C17.1, C18.2, C19.2, C20.2, C21.1, C22.1, C23.1, C24.1, C25.1, C26.1, C27.1, C28.1, C29.1, D1.1 (K), P1.5 (GND), P1.S1, P1.S2, P1.S3, P1.S4, P1.S5, P1.S6, R01.2, U1.3 (GND), U1.6 (TAB), U2.16 (GND), U2.6 (GND), U3.20 (AVSS), U3.25 (VSS), U3.35 (VSS), U3.40 (VSS), U3.55 (VSS), U3.59 (VSS), U3.7 (VSS)
- new net MCLR: U3.9 (*MCLR)
- new net OSC1: U3.31 (OSC1/CLKI/RC12)
- new net OSC2: U3.32 (OSC2/CLKO/RC15)
- new net PGEC2: U3.17 (PGEC2/AN46/RPB6/RB6)
- new net PGED2: U3.18 (PGED2/AN47/RPB7/RB7)
- new net RB0: U3.16 (PGED1/VREF+/CVREF+/AN0/RPB0/PMA6/RB0)
- new net RB1: U3.15 (PGEC1/VREF-/CVREF-/AN1/RPB1/RB1)
- new net RB10: U3.23 (TMS/CVREFOUT/AN5/RPB10/PMA13/RB10)
- new net RB11: U3.24 (TDO/AN6/PMA12/RB11)
- new net RB13: U3.28 (TDI/AN8/RB13)
- new net RB14: U3.29 (AN9/RPB14/SCK3/PMA1/RB14)
- new net RB15: U3.30 (AN10/EMDC/AEMDC/RPB15/OCFB/PMA0/RB15)
- new net RB2: U3.14 (AN2/C2INB/RPB2/RB2)
- new net RB3: U3.13 (AN3/C2INA/RPB3/RB3)
- new net RB4: U3.12 (AN4/C1INB/RB4)
- new net RB5: U3.11 (AN45/C1INA/RPB5/RB5)
- new net RB8: U3.21 (AN48/RPB8/PMA10/RB8)
- new net RB9: U3.22 (AN49/RPB9/PMA7/RB9)
- new net RD0: U3.46 (AERXD1/ETXD3/RPD0/RTCC/INT0/RD0)
- new net RD1: U3.49 (EMDIO/AEMDIO/RPD1/SCK1/RD1)
- new net RD10: U3.44 (ECOL/RPD10/SCL1/SCK4/RD10)
- new net RD11: U3.45 (AERXCLK/AEREFCLK/ECRS/RPD11/PMCS1/PMA14/RD11)
- new net RD2: U3.50 (ETXERR/AETXEN/RPD2/SDA3/RD2)
- new net RD3: U3.51 (AERXERR/ETXCLK/RPD3/SCL3/RD3)
- new net RD4: U3.52 (*SQICS0/RPD4/PMWR/RD4)
- new net RD9: U3.43 (AERXD0/ETXD2/RPD9/SDA1/PMCS2/PMA15/RD9)
- new net RE0: U3.58 (TRD0/SQID0/ERXD1/PMD0/RE0)
- new net RE1: U3.61 (TRD1/SQID1/ERXD0/PMD1/RE1)
- new net RE2: U3.62 (TRD2/SQID2/ERXDV/ECRSDV/AECRSDV/PMD2/RE2)
- new net RE3: U3.63 (TRD3/SQID3/ERXCLK/EREFCLK/RPE3/PMD3/RE3)
- new net RE4: U3.64 (AN18/ERXERR/PMD4/RE4)
- new net RE5: U3.1 (AN17/ETXEN/RPE5/PMD5/RE5)
- new net RE6: U3.2 (AN16/ETXD0/PMD6/RE6)
- new net RE7: U3.3 (AN15/ETXD1/PMD7/RE7)
- new net RF0: U3.56 (ERXD3/AETXD1/RPF0/RF0)
- new net RF1: U3.57 (TRCLK/SQICLK/ERXD2/AETXD0/RPF1/RF1)
- new net RF4: U3.41 (RPF4/SDA5/PMA9/RF4)
- new net RF5: U3.42 (RPF5/SCL5/PMA8/RF5)
- new net RG6: U3.4 (AN14/C1IND/RPG6/SCK2/PMA5/RG6)
- new net RG7: U3.5 (AN13/C1INC/RPG7/SDA4/PMA4/RG7)
- new net RG8: U3.6 (AN12/C2IND/RPG8/SCL4/PMA3/RG8)
- new net RG9: U3.10 (AN11/C2INC/RPG9/PMA2/RG9)
- new net SOSCI: U3.47 (SOSCI/RPC13/RC13)
- new net SOSCO: U3.48 (SOSCO/RPC14/T1CK/RC14)
- new net U1RX: U2.20 (TXD), U3.27 (TCK/AN7/PMA11/RB12)
- new net U1TX: U2.4 (RXD), U3.53 (*SQICS1/RPD5/PMRD/RD5)
- new net USBID: U3.38 (RPF3/USBID/RF3)
- new net VBUS: U3.33 (VBUS)
- no-connect marks 0 -> 11

Commit message: more
Parts:
- added C30, C31, C32, C33: 100n, Capacitor_SMD:C_0603_1608Metric_Pad1.08x0.95mm_HandSolder, symbol Device:C_Small
- added D2: LED_GREEN, symbol Lib:LED_GREEN
- added D3: LED_YELLOW, symbol Lib:LED_YELLOW
- added D4: LED_ORANGE, symbol Lib:LED_ORANGE
- added D5: LED_RED, symbol Lib:LED_RED
- added P2: Conn_01x08_Pin, Connector_PinHeader_1.00mm:PinHeader_1x08_P1.00mm_Horizontal, symbol Lib:Conn_01x08_Pin
- added P3: Conn_01x05_Pin, Connector_PinHeader_1.00mm:PinHeader_1x05_P1.00mm_Vertical, symbol Lib:Conn_01x05_Pin
- added P4: Conn_01x06_Pin, Connector_PinHeader_1.00mm:PinHeader_1x06_P1.00mm_Vertical, symbol Lib:Conn_01x06_Pin
- added P5: HSEC8-120-01-S-D-EM2, Lib_fp:SAMTEC_HSEC8-120-01-S-D-EM2, symbol Lib:HSEC8-120-01-S-D-EM2
- added R05, R06, R07, R09: 10K, Resistor_SMD:R_0603_1608Metric_Pad0.98x0.95mm_HandSolder, symbol Device:R_US
- added R08: 1K, Resistor_SMD:R_0603_1608Metric_Pad0.98x0.95mm_HandSolder, symbol Device:R_US
- added R10: 4K53, Resistor_SMD:R_0603_1608Metric_Pad0.98x0.95mm_HandSolder, symbol Device:R_US
- added R11: 470, Resistor_SMD:R_0603_1608Metric_Pad0.98x0.95mm_HandSolder, symbol Device:R_US
- added R12: 2K7, Resistor_SMD:R_0603_1608Metric_Pad0.98x0.95mm_HandSolder, symbol Device:R_US
- added R13: 1K37, Resistor_SMD:R_0603_1608Metric_Pad0.98x0.95mm_HandSolder, symbol Device:R_US
- added S1: B3F-1002, Lib_fp:SW_B3F-1000_OMR, symbol Lib:B3F-1002
- added S2: B3F-1000, Lib_fp:SW_B3F-1000_OMR, symbol Lib:B3F-1000
- added S3, S4: B3F-1005, Lib_fp:SW_B3F-1000_OMR, symbol Lib:B3F-1005
- U3: footprint TQFP64_PT_MCH -> Lib_fp:TQFP64_PT_MCH
Connections:
- net +3V3: now also D2.2 (A), P2.3 (Pin_3), P4.2 (Pin_2), R05.2, R06.2, R07.2, R09.2
- net +3V3AUX: now also P5.16, P5.39
- net +5VAUX: now also P5.40
- net D+: now also P4.4 (Pin_4)
- net D-: now also P4.3 (Pin_3)
- net GND: now also C30.2, C31.2, C32.2, C33.2, P2.2 (Pin_2), P3.3 (Pin_3), P4.6 (Pin_6), P5.02, P5.19, P5.33, P5.S1, P5.S2, P5.S3, P5.S4, R10.1, R11.1, R12.1, R13.1, S1.2, S1.4, S2.2, S2.4, S3.2, S3.4, S4.2, S4.4
- net MCLR: now also P2.1 (Pin_1), R08.2
- net OSC1: now also P3.1 (Pin_1)
- net OSC2: now also P3.2 (Pin_2)
- net PGEC2: now also P2.5 (Pin_5)
- net PGED2: now also P2.4 (Pin_4)
- net RB0: now also P5.11
- net RB1: now also P5.13
- net RB10: now also P5.07
- net RB11: now also P5.05
- net RB13: now also P5.03
- net RB14: now also D5.2 (A)
- net RB15: now also P5.01
- net RB2: now also P5.15
- net RB3: now also P5.17
- net RB4: now also P5.21
- net RB5: now also P5.23
- net RB8: now also P5.09
- net RB9: now also D4.2 (A)
- net RD0: now also P5.14
- net RD1: now also P5.18
- net RD10: now also P5.10
- net RD11: now also P5.12
- net RD2: now also P5.20
- net RD3: now also P5.22
- net RD4: now also P5.24
- net RD9: now also P5.08
- net RE0: now also P5.30
- net RE1: now also P5.32
- net RE2: now also P5.34
- net RE3: now also P5.36
- net RE4: now also P5.38
- net RE5: now also P5.37
- net RE6: now also P5.35
- net RE7: now also P5.31
- net RF0: now also P5.26
- net RF1: now also P5.28
- net RF4: now also P5.04
- net RF5: now also P5.06
- net RG6: now also C30.1, P5.29, R05.1, S1.1, S1.3
- net RG7: now also C31.1, P5.27, R06.1, S2.1, S2.3
- net RG8: now also C32.1, P5.25, R07.1, S3.1, S3.3
- net RG9: now also D3.2 (A)
- net SOSCI: now also P3.4 (Pin_4)
- net SOSCO: now also P3.5 (Pin_5)
- net USBID: now also P4.5 (Pin_5)
- net VBUS: now also P4.1 (Pin_1)
- new net: D4.1 (K), R12.2
- new net: D3.1 (K), R11.2
- new net: D5.1 (K), R13.2
- new net: C33.1, R08.1, R09.1, S4.1, S4.3
- new net: D2.1 (K), R10.2
- no-connect marks 11 -> 14

Commit message: update
Parts:
- D1, D2, D3, D4, D5: footprint (none) -> Lib_fp:LED_APT1608LVBC_D
- J1, J2: footprint (none) -> Connector_PinHeader_2.54mm:PinHeader_2x03_P2.54mm_Vertical
- P2: footprint Connector_PinHeader_1.00mm:PinHeader_1x08_P1.00mm_Horizontal -> Connector_PinHeader_2.54mm:PinHeader_1x08_P2.54mm_Horizontal
- P3: footprint Connector_PinHeader_1.00mm:PinHeader_1x05_P1.00mm_Vertical -> Connector_PinHeader_2.54mm:PinHeader_1x05_P2.54mm_Vertical
- P4: footprint Connector_PinHeader_1.00mm:PinHeader_1x06_P1.00mm_Vertical -> Connector_PinHeader_2.54mm:PinHeader_1x06_P2.54mm_Vertical
Changed lines of the file:
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@@
 			)
 		)
-		(property "Footprint" ""
+		(property "Footprint" "Lib_fp:LED_APT1608LVBC_D"
 			(at 234.95 176.53 0)
 			(effects
@@
 			)
 		)
-		(property "Footprint" ""
+		(property "Footprint" "Lib_fp:LED_APT1608LVBC_D"
 			(at 213.36 176.53 0)
 			(effects
@@
 			)
 		)
-		(property "Footprint" ""
+		(property "Footprint" "Connector_PinHeader_2.54mm:PinHeader_2x03_P2.54mm_Vertical"
 			(at 137.16 57.15 0)
 			(effects
@@
 			)
 		)
-		(property "Footprint" ""
+		(property "Footprint" "Connector_PinHeader_2.54mm:PinHeader_2x03_P2.54mm_Vertical"
 			(at 74.93 41.91 0)
 			(effects
@@
 			)
 		)
-		(property "Footprint" ""
+		(property "Footprint" "Lib_fp:LED_APT1608LVBC_D"
 			(at 106.68 133.35 0)
 			(effects
@@
 			)
 		)
-		(property "Footprint" "Connector_PinHeader_1.00mm:PinHeader_1x08_P1.00mm_Horizontal"
+		(property "Footprint" "Connector_PinHeader_2.54mm:PinHeader_1x08_P2.54mm_Horizontal"
 			(at 52.07 233.68 0)
 			(effects
@@
 			)
 		)
-		(property "Footprint" ""
+		(property "Footprint" "Lib_fp:LED_APT1608LVBC_D"
 			(at 256.54 176.53 0)
 			(effects
@@
 			)
 		)
-		(property "Footprint" "Connector_PinHeader_1.00mm:PinHeader_1x05_P1.00mm_Vertical"
+		(property "Footprint" "Connector_PinHeader_2.54mm:PinHeader_1x05_P2.54mm_Vertical"
 			(at 97.79 226.06 0)
 			(effects
@@
 			)
 		)
-		(property "Footprint" ""
+		(property "Footprint" "Lib_fp:LED_APT1608LVBC_D"
 			(at 191.77 176.53 0)
 			(effects
@@
 			)
 		)
-		(property "Footprint" "Connector_PinHeader_1.00mm:PinHeader_1x06_P1.00mm_Vertical"
+		(property "Footprint" "Connector_PinHeader_2.54mm:PinHeader_1x06_P2.54mm_Vertical"
 			(at 128.27 226.06 0)
 			(effects
