File: Projeto2/Projeto2.kicad_pcb (KiCad board)
At the start: 2 copper layers, 54 x 54 mm, 12 parts, among them P1 10118194-0001LF, P2 Conn_01x08_Pin, P3 Conn_01x05_Pin, P4 Conn_01x06_Pin, P5 HSEC8-120-01-S-D-EM2, U1 TPS79633DCQR, U2 FT231XS-R, U3 PIC32MZ1024EFE064-E/PT

Commit message: update
Parts:
- added C02: 10n, Capacitor_SMD:C_0805_2012Metric_Pad1.18x1.45mm_HandSolder, F.Cu at (211.7, 76.3)
- added C03: 1u, Capacitor_SMD:C_0805_2012Metric_Pad1.18x1.45mm_HandSolder, F.Cu at (211.7, 79.3)
- added C04: 10n, Capacitor_SMD:C_0805_2012Metric_Pad1.18x1.45mm_HandSolder, F.Cu at (211.7, 82.3)
- added C05: 47p, Capacitor_SMD:C_0805_2012Metric_Pad1.18x1.45mm_HandSolder, F.Cu at (216.5, 73.3)
- added C06: 47p, Capacitor_SMD:C_0805_2012Metric_Pad1.18x1.45mm_HandSolder, F.Cu at (216.5, 76.3)
- added C07: 4u7, Capacitor_SMD:C_0603_1608Metric_Pad1.08x0.95mm_HandSolder, F.Cu at (211.4, 55.4)
- added C08: 100n, Capacitor_SMD:C_0603_1608Metric_Pad1.08x0.95mm_HandSolder, F.Cu at (211.4, 58.0)
- added C09: 100n, Capacitor_SMD:C_0603_1608Metric_Pad1.08x0.95mm_HandSolder, F.Cu at (211.4, 60.5)
- added C1: 2u2, Capacitor_SMD:C_0805_2012Metric_Pad1.18x1.45mm_HandSolder, F.Cu at (211.7, 73.3)
- added C10: 10u, Capacitor_SMD:C_0805_2012Metric_Pad1.18x1.45mm_HandSolder, F.Cu at (216.5, 79.3)
- added C11: 100n, Capacitor_SMD:C_0603_1608Metric_Pad1.08x0.95mm_HandSolder, F.Cu at (211.4, 63.0)
- added C12: 10n, Capacitor_SMD:C_0603_1608Metric_Pad1.08x0.95mm_HandSolder, F.Cu at (211.4, 65.5)
- added C13: 100n, Capacitor_SMD:C_0603_1608Metric_Pad1.08x0.95mm_HandSolder, F.Cu at (211.4, 68.0)
- added C14: 10n, Capacitor_SMD:C_0603_1608Metric_Pad1.08x0.95mm_HandSolder, F.Cu at (211.4, 70.5)
- added C15: 10u, Capacitor_SMD:C_0805_2012Metric_Pad1.18x1.45mm_HandSolder, F.Cu at (216.5, 82.3)
- added C16: 100n, Capacitor_SMD:C_0603_1608Metric_Pad1.08x0.95mm_HandSolder, F.Cu at (215.8, 55.4)
- added C17: 10n, Capacitor_SMD:C_0603_1608Metric_Pad1.08x0.95mm_HandSolder, F.Cu at (215.8, 58.0)
- added C18: 10n, Capacitor_SMD:C_0603_1608Metric_Pad1.08x0.95mm_HandSolder, F.Cu at (215.8, 60.5)
- added C19: 100n, Capacitor_SMD:C_0603_1608Metric_Pad1.08x0.95mm_HandSolder, F.Cu at (215.8, 63.0)
- added C20: 10u, Capacitor_SMD:C_0805_2012Metric_Pad1.18x1.45mm_HandSolder, F.Cu at (221.3, 73.3)
- added C21: 10n, Capacitor_SMD:C_0603_1608Metric_Pad1.08x0.95mm_HandSolder, F.Cu at (215.8, 65.5)
- added C22: 100n, Capacitor_SMD:C_0603_1608Metric_Pad1.08x0.95mm_HandSolder, F.Cu at (215.8, 68.0)
- added C23: 10u, Capacitor_SMD:C_0805_2012Metric_Pad1.18x1.45mm_HandSolder, F.Cu at (221.3, 76.3)
- added C24: 10n, Capacitor_SMD:C_0603_1608Metric_Pad1.08x0.95mm_HandSolder, F.Cu at (160.8, 90.2)
- added C25: 100n, Capacitor_SMD:C_0603_1608Metric_Pad1.08x0.95mm_HandSolder, F.Cu at (159.7, 89.2)
- added C26: 10u, Capacitor_SMD:C_0805_2012Metric_Pad1.18x1.45mm_HandSolder, F.Cu at (158.4, 87.9)
- added C27: 10n, Capacitor_SMD:C_0603_1608Metric_Pad1.08x0.95mm_HandSolder, F.Cu at (163.5, 87.5)
- added C28: 100n, Capacitor_SMD:C_0603_1608Metric_Pad1.08x0.95mm_HandSolder, F.Cu at (162.4, 86.4)
- added C29: 10u, Capacitor_SMD:C_0805_2012Metric_Pad1.18x1.45mm_HandSolder, F.Cu at (161.1, 85.2)
- added C30: 100n, Capacitor_SMD:C_0603_1608Metric_Pad1.08x0.95mm_HandSolder, F.Cu at (220.1, 63.0)
- added C31: 100n, Capacitor_SMD:C_0603_1608Metric_Pad1.08x0.95mm_HandSolder, F.Cu at (220.1, 65.5)
- added C32: 100n, Capacitor_SMD:C_0603_1608Metric_Pad1.08x0.95mm_HandSolder, F.Cu at (220.1, 68.0)
- added C33: 100n, Capacitor_SMD:C_0603_1608Metric_Pad1.08x0.95mm_HandSolder, F.Cu at (220.1, 70.5)
- added L1: FerriteBead_Small, Inductor_SMD:L_0603_1608Metric_Pad1.05x0.95mm_HandSolder, F.Cu at (224.5, 55.4)
- added L2: 0.2n, Inductor_SMD:L_0402_1005Metric_Pad0.77x0.64mm_HandSolder, F.Cu at (225.3, 72.8)
- added R01: 1k, Resistor_SMD:R_0603_1608Metric_Pad0.98x0.95mm_HandSolder, F.Cu at (224.5, 58.0)
- added R03: 27, Resistor_SMD:R_0603_1608Metric_Pad0.98x0.95mm_HandSolder, F.Cu at (224.5, 63.0)
- added R04: 27, Resistor_SMD:R_0603_1608Metric_Pad0.98x0.95mm_HandSolder, F.Cu at (224.5, 65.5)
- added R05: 10K, Resistor_SMD:R_0603_1608Metric_Pad0.98x0.95mm_HandSolder, F.Cu at (224.5, 68.0)
- added R06: 10K, Resistor_SMD:R_0603_1608Metric_Pad0.98x0.95mm_HandSolder, F.Cu at (224.5, 70.5)
- added R07: 10K, Resistor_SMD:R_0603_1608Metric_Pad0.98x0.95mm_HandSolder, F.Cu at (228.8, 55.4)
- added R08: 1K, Resistor_SMD:R_0603_1608Metric_Pad0.98x0.95mm_HandSolder, F.Cu at (228.8, 58.0)
- added R09: 10K, Resistor_SMD:R_0603_1608Metric_Pad0.98x0.95mm_HandSolder, F.Cu at (228.8, 60.5)
- added R10: 4K53, Resistor_SMD:R_0603_1608Metric_Pad0.98x0.95mm_HandSolder, F.Cu at (228.8, 63.0)
- added R11: 470, Resistor_SMD:R_0603_1608Metric_Pad0.98x0.95mm_HandSolder, F.Cu at (228.8, 65.5)
- added R12: 2K7, Resistor_SMD:R_0603_1608Metric_Pad0.98x0.95mm_HandSolder, F.Cu at (228.8, 68.0)
- added R13: 1K37, Resistor_SMD:R_0603_1608Metric_Pad0.98x0.95mm_HandSolder, F.Cu at (228.8, 70.5)
- added R2: 1k, Resistor_SMD:R_0603_1608Metric_Pad0.98x0.95mm_HandSolder, F.Cu at (224.5, 60.5)
- moved P3 1.24 mm to (156.5, 86.5)
- moved P5 0.91 mm to (185.7, 95.4)
- moved S4 0.79 mm to (173.9, 77.5)
- moved S3 0.40 mm to (176.0, 119.8)
- moved P2 0.30 mm to (162.0, 72.7)
Other:
- outline, holes or cut-outs redrawn
- copper layers 2 -> 4

Commit message: update
Parts:
- added D1: LED_BLUE, Lib_fp:LED_APT1608LVBC_D, F.Cu at (148.5, 91.8)
- added D2: LED_GREEN, Lib_fp:LED_APT1608LVBC_D, F.Cu at (175.6, 101.2)
- added D3: LED_YELLOW, Lib_fp:LED_APT1608LVBC_D, F.Cu at (176.7, 108.9)
- added D4: LED_ORANGE, Lib_fp:LED_APT1608LVBC_D, F.Cu at (179.7, 108.9)
- added D5: LED_RED, Lib_fp:LED_APT1608LVBC_D, F.Cu at (173.7, 108.9)
- added J1: Conn_02x03_Odd_Even, Connector_PinHeader_2.54mm:PinHeader_2x03_P2.54mm_Vertical, F.Cu at (147.3, 119.0)
- added J2: Conn_02x03_Odd_Even, Connector_PinHeader_2.54mm:PinHeader_2x03_P2.54mm_Vertical, F.Cu at (151.1, 80.3)
- added REF**: MountingHole_3.2mm_M3_ISO14580_Pad, MountingHole:MountingHole_3.2mm_M3_ISO14580_Pad, F.Cu at (185.5, 118.0)
- added REF**: MountingHole_3.2mm_M3_ISO14580_Pad, MountingHole:MountingHole_3.2mm_M3_ISO14580_Pad, F.Cu at (141.5, 118.0)
- added REF**: MountingHole_3.2mm_M3_ISO14580_Pad, MountingHole:MountingHole_3.2mm_M3_ISO14580_Pad, F.Cu at (185.5, 74.0)
- added REF**: MountingHole_3.2mm_M3_ISO14580_Pad, MountingHole:MountingHole_3.2mm_M3_ISO14580_Pad, F.Cu at (141.5, 74.0)
- P2: footprint Connector_PinHeader_1.00mm:PinHeader_1x08_P1.00mm_Horizontal -> Connector_PinHeader_2.54mm:PinHeader_1x08_P2.54mm_Horizontal
- P3: footprint Connector_PinHeader_1.00mm:PinHeader_1x05_P1.00mm_Vertical -> Connector_PinHeader_2.54mm:PinHeader_1x05_P2.54mm_Vertical
- P4: footprint Connector_PinHeader_1.00mm:PinHeader_1x06_P1.00mm_Vertical -> Connector_PinHeader_2.54mm:PinHeader_1x06_P2.54mm_Vertical
- moved R01 96.4 mm to (145.2, 112.8)
- moved L1 88.1 mm to (143.5, 90.2), turned to 180 degrees
- moved R2 85.3 mm to (145.2, 91.8), turned to 180 degrees
- moved R04 84.5 mm to (146.0, 96.9), turned to 90 degrees
- moved R03 82.2 mm to (149.7, 96.9), turned to 90 degrees
- moved C30 80.2 mm to (157.2, 112.7)
- moved R05 78.0 mm to (160.6, 112.7)
- moved C06 75.2 mm to (144.2, 97.0), turned to 90 degrees
- moved R07 74.9 mm to (180.3, 112.5)
- moved C07 73.3 mm to (146.9, 90.2), turned to 180 degrees
- moved C05 72.6 mm to (147.8, 96.9), turned to 90 degrees
- moved R06 71.4 mm to (166.8, 112.6)
- moved C08 71.4 mm to (146.9, 88.6), turned to 180 degrees
- moved C04 71.3 mm to (140.7, 89.7), turned to -90 degrees
- moved C1 70.7 mm to (150.4, 108.5), turned to 90 degrees
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Other:
- outline, holes or cut-outs redrawn

Commit message: another one
Parts:
- added 3V3: TestPoint_Pad_D1.5mm, TestPoint:TestPoint_Pad_D1.5mm, F.Cu at (158.0, 77.5)
- added 5V: TestPoint_Pad_D1.5mm, TestPoint:TestPoint_Pad_D1.5mm, F.Cu at (155.0, 108.0)
- added GND: TestPoint_Pad_D1.5mm, TestPoint:TestPoint_Pad_D1.5mm, F.Cu at (169.0, 77.5)
- moved C09 2.40 mm to (142.0, 79.9)
- moved U2 1.78 mm to (142.6, 84.2)
- moved J2 1.61 mm to (149.5, 80.5)
- moved P1 1.53 mm to (139.5, 97.5)
Connections:
- REF** pad 1: (no net) -> GND (x4)
Routing:
- net +3V3: track 0.00 -> 156.8 mm
- net +5V0USB: track 0.00 -> 61.8 mm
- net +5VAUX: track 0.00 -> 42.1 mm
- net U1RX: track 0.00 -> 38.3 mm, vias 0 -> 2
- net MCLR: track 0.00 -> 38.1 mm
- net U1TX: track 0.00 -> 31.3 mm, vias 0 -> 2
- net RG6: track 0.00 -> 26.7 mm
- net RG7: track 0.00 -> 22.7 mm
- net Net-(U2-USBDP): track 0.00 -> 20.6 mm, vias 0 -> 2
- net +5V: track 0.00 -> 19.8 mm
- net Net-(U2-USBDM): track 0.00 -> 18.7 mm, vias 0 -> 2
- net RG8: track 0.00 -> 18.3 mm
- net Net-(J2-Pin_3): track 0.00 -> 16.2 mm, vias 0 -> 2
- net Net-(P1-VCC): track 0.00 -> 14.2 mm
- net Net-(C33-Pad1): track 0.00 -> 12.3 mm
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- added copper zone on B.Cu, net GND
- added copper zone on F.Cu, net GND

Commit message: project 2 done
Parts:
- moved D5 3.20 mm to (170.5, 109.1)
- moved R13 2.31 mm to (172.9, 109.1)
- moved C32 1.91 mm to (175.2, 111.6)
- moved C30 1.89 mm to (155.5, 111.8)
- moved R05 1.73 mm to (159.1, 111.8)
- moved D3 1.71 mm to (175.0, 109.1)
- moved D2 1.58 mm to (176.8, 102.3)
- moved C1 1.18 mm to (151.6, 108.5)
- moved R11 1.00 mm to (177.2, 109.0)
- moved C06 0.83 mm to (144.2, 97.8)
- moved R01 0.80 mm to (144.4, 112.8)
- moved D4 0.10 mm to (179.6, 108.9)
Connections:
- P1 pad SH1: (no net) -> GND
- P1 pad SH2: (no net) -> GND
- P1 pad SH3: (no net) -> GND
- P1 pad SH4: (no net) -> GND
- P1 pad SH5: (no net) -> GND
- P1 pad SH6: (no net) -> GND
- U1 pad 10: (no net) -> GND
- U1 pad 11: (no net) -> GND
- U1 pad 12: (no net) -> GND
- U1 pad 13: (no net) -> GND
- U1 pad 14: (no net) -> GND
- U1 pad 15: (no net) -> GND
- U1 pad 16: (no net) -> GND
- U1 pad 7: (no net) -> GND
- U1 pad 8: (no net) -> GND
- U1 pad 9: (no net) -> GND
Routing:
- net GND: track 0.00 -> 166.8 mm, vias 0 -> 34
- net +3V3AUX: track 0.00 -> 111.8 mm, vias 0 -> 3
- net +3V3: track 156.8 -> 255.6 mm, vias 0 -> 1
- net RG6: track 26.7 -> 82.7 mm, vias 0 -> 4
- net RG8: track 18.3 -> 71.0 mm, vias 0 -> 2
- net RG7: track 22.7 -> 65.4 mm, vias 0 -> 3
- net RE0: track 0.00 -> 36.4 mm, vias 0 -> 2
- net RD4: track 0.00 -> 36.2 mm, vias 0 -> 2
- net RD10: track 0.00 -> 34.2 mm, vias 0 -> 2
- net RE1: track 0.00 -> 33.8 mm, vias 0 -> 2
- net RE2: track 0.00 -> 33.4 mm, vias 0 -> 1
- net MCLR: track 38.1 -> 71.5 mm, vias 0 -> 1
- net RE4: track 0.00 -> 31.3 mm, vias 0 -> 2
- net RF5: track 0.00 -> 31.2 mm, vias 0 -> 2
- net RF1: track 0.00 -> 30.4 mm, vias 0 -> 1
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